File: assets/PCB Files/POSHA.kicad_sch (KiCad schematic)
At the start: 43 parts, among them J1 Battery Input, J2 Battery Input, J3 Battery Input, J4 Screw_Terminal_01x04, J5 Screw_Terminal_01x03, J6 Screw_Terminal_01x05, J7 Screw_Terminal_01x05, J8 Load Cell Input, J9 Screw_Terminal_01x04, SW1 SW_Push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

Commit message: Added PCB Files
Parts:
- removed R5, R6: 4.7k, symbol Device:R
- removed Rfbt1: 100k, symbol Device:R
- added R12: 100k, Resistor_SMD:R_1210_3225Metric_Pad1.30x2.65mm_HandSolder, symbol Device:R
- added R13, R14: 4.7k, Resistor_SMD:R_1210_3225Metric, symbol Device:R
- C1, C2, C3: footprint (none) -> Capacitor_SMD:C_2220_5750Metric_Pad1.97x5.40mm_HandSolder
- C4, C5, C6, Cboot1, Cff1, Chf1, Cin1, Cout1, Cvcc1: footprint (none) -> Capacitor_SMD:C_0201_0603Metric
- J1, J2, J3: footprint XT30PW-M:AMASS_XT30PW-M -> Connector_AMASS:AMASS_XT30U-F_1x02_P5.0mm_Vertical
- J4, J9: footprint (none) -> TerminalBlock:TerminalBlock_MaiXu_MX126-5.0-04P_1x04_P5.00mm
- J5: footprint (none) -> TerminalBlock:TerminalBlock_MaiXu_MX126-5.0-03P_1x03_P5.00mm
- J6: footprint (none) -> Connector_PinHeader_1.00mm:PinHeader_1x05_P1.00mm_Vertical
- J7: footprint (none) -> TerminalBlock:TerminalBlock_MaiXu_MX126-5.0-05P_1x05_P5.00mm
- L1, L2: footprint (none) -> Inductor_SMD:L_Neosid_SM-NE127_HandSoldering
- MotorConnect1: renamed from MotorConnect; footprint (none) -> TerminalBlock:TerminalBlock_MaiXu_MX126-5.0-03P_1x03_P5.00mm
- R1, R11: footprint (none) -> Resistor_SMD:R_1210_3225Metric_Pad1.30x2.65mm_HandSolder
- R10, R7, R8, R9: footprint (none) -> Resistor_SMD:R_1210_3225Metric
- R2: footprint (none) -> Resistor_SMD:R_01005_0402Metric
- R3, R4: footprint (none) -> Resistor_SMD:R_0201_0603Metric
- Rfbb1: footprint (none) -> Resistor_SMD:R_0805_2012Metric
- SW1: footprint (none) -> Button_Switch_THT:SW_PUSH_1P1T_6x3.5mm_H5.0_APEM_MJTP1250
- U1: footprint (none) -> Teensy:Teensy41
Connections:
- net +3.3V: now also R10.2, R9.2, R13.1, R14.1; no longer R10.1, R9.1
- net +5V: now also R12.2
- net GND: now also J1.2, J2.1, J3.2; no longer J1.N, J2.P, J3.N
- net at C1.1, C2.1, C3.1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: now also J3.1; no longer J3.P
- net at C5.1, Chf1.1, Cin1.1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: now also J1.1, J2.2; no longer J1.P, J2.N
- net at U1.17 (25_A11_RX6_SDA2), U4.3 (SDA): now also R14.2
- net at U1.16 (24_A10_TX6_SCL2), U4.4 (SCL): now also R13.2
- net at Cff1.2, Rfbb1.1, U2.5 (FB): now also R12.1
- net at J9.4 (Pin_4), U1.38 (16_A2_RX4_SCL1): now also R9.1; no longer R10.2
- net at J9.3 (Pin_3), U1.39 (17_A3_TX4_SDA1): now also R10.1; no longer R9.2
- no-connect marks 1 -> 61
